Commit message: [ADD] Gazebo tag in urdf file
Step 3.7 in document:
file:///C:/Users/HH/OneDrive/3_Research/EndNote_Library/5_Etc/Importing_URDF_Package_from_Soloidworks_in_ROS.pdf

File: Dual_arm_ws/src/dual_arm_hh/urdf/dual_arm_urdf.urdf (robot description, URDF)
Before this commit: robot Dual_arm_HH, 11 links, 10 joints
Joints:
- joint Joint_1_left: limit (none) -> lower=-3.142 upper=3.142 effort=300 velocity=3; type continuous -> revolute
- joint Joint_1_right: limit (none) -> lower=-3.142 upper=3.142 effort=300 velocity=3; type continuous -> revolute
- joint Joint_2_left: limit (none) -> lower=-3.142 upper=3.142 effort=300 velocity=3; type continuous -> revolute
- joint Joint_2_right: limit (none) -> lower=-3.142 upper=3.142 effort=300 velocity=3; type continuous -> revolute
- joint Joint_3_left: limit (none) -> lower=-3.142 upper=3.142 effort=300 velocity=3; type continuous -> revolute
- joint Joint_3_right: limit (none) -> lower=-3.142 upper=3.142 effort=300 velocity=3; type continuous -> revolute

Commit message: [FIX] dual arm urdf doesn't load correctly in gazebo
(problem)
 - Link_0_right  has no inertia and mass, which make the next link cannot connect to it
 - Note that NO error is pop-up in terminal when launching it

(solve) Copy inertia and mass of Link_0_left for Link_0_right

(mod) Mod the .urdf file for increasing readability

File: Dual_arm_ws/src/dual_arm_hh/urdf/dual_arm_urdf.urdf (robot description, URDF)
Before this commit: robot Dual_arm_HH, 11 links, 10 joints
Links:
- link Link_0_right: mass 0 -> 44.0003903821512
Joints:
- joint Joint_1_left: origin xyz=0.18 0.475 -0.0875 rpy=0 0 0 -> xyz=0.18 0.475 -0.0875 rpy=0 0 1.5708
- joint Joint_1_right: axis 0 0 -1 -> 0 0 1; origin xyz=0.18 0.475 -0.0875 rpy=0 0 0 -> xyz=0.18 0.475 -0.0875 rpy=0 0 1.5708
- joint Joint_2_right: axis 0 0 -1 -> 0 0 1
- joint Joint_3_right: axis 0 0 -1 -> 0 0 1
- joint base_joint: origin xyz=0.0 0.0 0.17 rpy=0 0 0 -> xyz=0 0 0 rpy=0 0 0

Commit message: [MOD] init position of dual-arm [ADD] result video
[MOD] init position of dual-arm
init position is the arm make a line parallel with the horizontal

[ADD] result video
video for cosim_trajectory_no_object

NOTE: Now it can work with Simulink file "Cosim_03_Dual_arm_Planning.slx"
TODO: Add plannar joint for Object and control it

File: Dual_arm_ws/src/dual_arm_hh/urdf/dual_arm_urdf.urdf (robot description, URDF)
Before this commit: robot Dual_arm_HH, 11 links, 10 joints
Joints:
- joint Joint_1_left: origin xyz=0.18 0.475 -0.0875 rpy=0 0 1.5708 -> xyz=0.18 0.475 -0.0875 rpy=0 0 0
- joint Joint_1_right: origin xyz=0.18 0.475 -0.0875 rpy=0 0 1.5708 -> xyz=0.18 0.475 -0.0875 rpy=0 0 0

Commit message: [MOD] Camera Pose [MOD] Plugin syntax [ADD] Collide tag [MOD] Init Pose
Note: this is end of position control without object
Mod:
 - Camera pose for better view
 - Enable collide feature
 - Adjust robot init pose for avoiding collision
 - Mode Cosim plugin tag increasing readability

File: Dual_arm_ws/src/dual_arm_hh/urdf/dual_arm_urdf.urdf (robot description, URDF)
Before this commit: robot Dual_arm_HH, 11 links, 10 joints
Links:
- removed link Link_object
Joints:
- removed joint Joint_0_object
- joint Joint_1_left: origin xyz=0.18 0.475 -0.0875 rpy=0 0 0 -> xyz=0.18 0.475 -0.0875 rpy=0 0 1.5708
- joint Joint_1_right: origin xyz=0.18 0.475 -0.0875 rpy=0 0 0 -> xyz=0.18 0.475 -0.0875 rpy=0 0 1.5708
