Commit message: [MOD] Chinh lai urdf
* dual_arm_hh package
 - ...force_urdf:
   + gom cac joint lai voi nhau
   + them damping va friction
   + tat collision

* dual_arm_left package
- ...left.urdf:
   + tang gioi han toc do va torque
   + them damping va friction
   + tat collision

File: Dual_arm_ws/src/dual_arm_hh/urdf/dual_arm_force_urdf.urdf (robot description, URDF)
Before this commit: robot Dual_arm_HH, 10 links, 9 joints
Joints:
- joint Joint_1_left: limit lower=-3.142 upper=3.142 effort=300 velocity=3 -> lower=-3.142 upper=3.142 effort=500 velocity=12.56; origin xyz=0.18 0.475 -0.0875 rpy=0 0 1.5708 -> xyz=0.18 0.475 -0.0875 rpy=0 0 0
- joint Joint_1_right: limit lower=-3.142 upper=3.142 effort=300 velocity=3 -> lower=-3.142 upper=3.142 effort=500 velocity=12.56; origin xyz=0.18 0.475 -0.0875 rpy=0 0 1.5708 -> xyz=0.18 0.475 -0.0875 rpy=0 0 0
- joint Joint_2_left: limit lower=-3.142 upper=3.142 effort=300 velocity=3 -> lower=-3.142 upper=3.142 effort=300 velocity=12.56
- joint Joint_2_right: limit lower=-3.142 upper=3.142 effort=300 velocity=3 -> lower=-3.142 upper=3.142 effort=300 velocity=12.56
- joint Joint_3_left: limit lower=-3.142 upper=3.142 effort=300 velocity=3 -> lower=-3.142 upper=3.142 effort=100 velocity=12.56
- joint Joint_3_right: limit lower=-3.142 upper=3.142 effort=300 velocity=3 -> lower=-3.142 upper=3.142 effort=100 velocity=12.56

File: Dual_arm_ws/src/dual_arm_left/urdf/dual_arm_left.urdf (robot description, URDF)
Before this commit: robot dual_arm_left, 6 links, 5 joints
Joints:
- joint joint_1: limit lower=-3.14 upper=3.14 effort=500 velocity=12.56 -> lower=-3.14 upper=3.14 effort=5000 velocity=120.56
- joint joint_2: limit lower=-3.14 upper=3.14 effort=300 velocity=12.56 -> lower=-3.14 upper=3.14 effort=3000 velocity=120.56
- joint joint_3: limit lower=-3.14 upper=3.14 effort=100 velocity=12.56 -> lower=-3.14 upper=3.14 effort=1000 velocity=120.56
