Commit message: [ADD] Init pose for MG  robot V10 [MOD] Friction and Gazebo view

File: Dual_arm_MG_ws/src/dual_arm/urdf/dual_arm_effort_position.xacro (robot description, xacro)
@@ -329,5 +329,5 @@
     <axis
       xyz="0 0 -1" />
-    <dynamics damping="0.05" friction="0.05"/>
+    <dynamics damping="0.05" friction="0.2"/>
     <limit
       lower="${-pi}"
@@ -380,5 +380,5 @@
     <axis
       xyz="0 0 1" />
-    <dynamics damping="0.05" friction="0.05"/>
+    <dynamics damping="0.05" friction="0.2"/>
     <limit
       lower="${-pi}"
@@ -431,5 +431,5 @@
     <axis
       xyz="0 0 -1" />
-    <dynamics damping="0.2" friction="0.1"/>
+    <dynamics damping="0.2" friction="0.4"/>
     <limit
       lower="${-pi}"
